Commit message: making ar tag bigger

File: urdf/ar_0.urdf (robot description, URDF)
Before this commit: robot ar_0, 1 links, 0 joints
Links:
- link ar_0: mass 0.00036 -> 0.00144; geometry collision box size=0.2 0.2 0.0001; visual mesh filename=package://ar_tags/meshes/MarkerData_0.dae

Commit message: making tag thicker

File: urdf/ar_0.urdf (robot description, URDF)
Before this commit: robot ar_0, 1 links, 0 joints
Links:
- link ar_0: geometry collision box size=0.2 0.2 0.01; visual mesh filename=package://ar_tags/meshes/MarkerData_0.dae
